Commit message: feat(ros): the description can wear the v6.27 legs
wojtek_body takes legs:=stock (default) or legs:=legs_v627, and the sim
xacro passes it through. Both leg macros use the same link and joint
names, so the ros2_control joint list and TF frames do not change. The
stock URDF expands identical to before; the new one matches the CAD
export's robot.urdf to 7e-9 in link poses, with the same joint limits.

The policy runtime reads the two contract fields such a policy brings: a
height table with its own third-joint column and a sign per leg, and a
null knee_singularity. It refuses clamp_knee for a policy without one.
The real launch sets clamp_knee, so a legs_v627 policy does not load on
the robot until someone decides that on purpose.

wojtek_real.urdf.xacro is untouched. A MuJoCo plant on these legs still
needs its scene and an identity joint map wired through the launch.

Co-Authored-By: Claude Fable 5.1 <noreply@anthropic.com>

File: ros/src/wojtek_description/urdf/body.urdf.xacro (robot description, xacro)
@@ -3,4 +3,5 @@
   <xacro:include filename="$(find wojtek_description)/urdf/inertia.urdf.xacro" />
   <xacro:include filename="$(find wojtek_description)/urdf/leg.urdf.xacro" />
+  <xacro:include filename="$(find wojtek_description)/urdf/leg_v627.urdf.xacro" />
   <!-- Mechanical assembly shared by every bringup of this robot: material,
        base_link/body_link/imu_link, and the four legs. ros2_control/Gazebo
@@ -13,6 +14,11 @@
        robot model owns the ground-truth extrinsics (machinekind/wojtek#91).
        The mount numbers must match wojtek_pc/camera_spec.py (MOUNT_XYZ,
-       MOUNT_PITCH_RAD); a test cross-checks them. -->
-  <xacro:macro name="wojtek_body" params="with_camera:=false">
+       MOUNT_PITCH_RAD); a test cross-checks them.
+       legs picks the set of legs bolted to this body: "stock" (the robot as
+       built, leg.urdf.xacro) or "legs_v627" (leg_v627.urdf.xacro, simulation
+       only so far). Both use the same link and joint names. The names match
+       training's robot variants (training/wojtek_rl/robots.py), where the
+       stock legs are called "wojtek". -->
+  <xacro:macro name="wojtek_body" params="with_camera:=false legs:=stock">
     <material name="grey">
       <color rgba="0.5 0.5 0.5 1" />
@@ -103,4 +109,5 @@
       </joint>
     </xacro:if>
+    <xacro:if value="${legs == 'stock'}">
     <xacro:leg prefix="rear_left" xyz="-0.131 0.06 0.06" rpy="0 0 ${pi}" first_joint_offset="${pi}"
       third_joint_gear_correction_dir="-1.0" />
@@ -112,4 +119,18 @@
       third_joint_gear_correction_dir="1.0"
     />
+    </xacro:if>
+    <xacro:if value="${legs == 'legs_v627'}">
+      <xacro:leg_v627 prefix="rear_left" xyz="-0.131 0.06 0.06" rpy="0 0 ${pi}"
+        first_joint_offset="${pi}" dir="-1.0" side="1.0" rear="true" />
+      <xacro:leg_v627 prefix="rear_right" xyz="-0.131 -0.06 0.06" rpy="0 0 ${pi}"
+        first_joint_offset="0.0" dir="1.0" side="-1.0" rear="true" />
+      <xacro:leg_v627 prefix="front_right" xyz="0.131 -0.06 0.06" rpy="0 0 0"
+        first_joint_offset="${pi}" dir="-1.0" side="-1.0" rear="false" />
+      <xacro:leg_v627 prefix="front_left" xyz="0.131 0.06 0.06" rpy="0 0 0"
+        first_joint_offset="0.0" dir="1.0" side="1.0" rear="false" />
+    </xacro:if>
+    <xacro:unless value="${legs in ('stock', 'legs_v627')}">
+      ${xacro.fatal("wojtek_body: legs must be 'stock' or 'legs_v627', got '" + legs + "'")}
+    </xacro:unless>
   </xacro:macro>
 </robot>

File: ros/src/wojtek_pc/urdf/wojtek_sim.urdf.xacro (robot description, xacro)
@@ -42,8 +42,14 @@
        gyro, so this is a plumbing switch, not a way to walk. -->
   <xacro:arg name="use_imu" default="true" />
+  <!-- Which legs the description shows: "stock" or "legs_v627" (see
+       wojtek_description's body.urdf.xacro). This swaps the URDF only. A
+       mujoco plant on the other legs also needs their scene as model_xml
+       (wojtek_description/mujoco/legs_v627/scene_mjx.xml) and an identity
+       joint map; that wiring does not exist yet. -->
+  <xacro:arg name="legs" default="stock" />
   <!-- In sim the robot model owns the camera extrinsics (ground truth) -
        robot_state_publisher latches base_link->camera_link->optical frames
        matching the MJCF render camera; see wojtek_pc/camera_spec.py. -->
-  <xacro:wojtek_body with_camera="true" />
+  <xacro:wojtek_body with_camera="true" legs="$(arg legs)" />
   <!-- Same interface set as wojtek_bringup's wojtek_joint macro: a position
        command (impedance target) and position/velocity/effort states. The
