Commit message: fix(ros): detect a dead drive link in md80_hardware_interface, restart via watchdog
When the SPI link or the CAN bus died under a live stack, nothing noticed:
the CANdle library only overwrites an Md80's state on a frame with that
drive's id and reports nothing when frames stop, read() copied the frozen
state and returned OK, the controllers stayed "active" and joint_states kept
publishing the last good sample (2026-09-21: motor power cycled under a live
stack, robot deaf for 30 min while every status was green). The on-robot
watchdog only knew a dead ros2_control_node or the bring-up-time "No answer"
log line, so it had nothing to react to.

Driver: a LinkMonitor per drive, hooked into the library's per-drive RX
callback, counts accepted frames; read() fails once any drive delivered no
frame for more than link_timeout_cycles cycles (new <hardware> param, 20 =
100 ms in the xacro, 0 = off). The controller manager then deactivates the
controllers and calls on_error, which stops the CANdle update loop and
leaves the component unconfigured. gtest for the monitor.

Watchdog: versioned under ros/deploy/rpi (it lived only on the robot) and
installed by install.sh phase 5. It now also watches the component state on
/controller_manager/activity: a non-active MD80HardwareInterface or a dead
CM stops the service, then mdtool probes the drives and the service starts
again once they answer -- no restart-looping while motor power is off.

Co-Authored-By: Claude Fable 5.1 <noreply@anthropic.com>

File: ros/src/wojtek_bringup/urdf/wojtek_ros2_control.urdf.xacro (robot description, xacro)
@@ -50,5 +50,5 @@
        8 since the 2026-07-17 migration for the HAT; the dongle setup ran 1.
        See ros/hw_tests/README.md for the per-drive baud migration tool. -->
-  <xacro:macro name="wojtek_ros2_control" params="kp kd max_torque usb_port bus:=spi can_baud:=8 dry_run:=false tau_ff:=false">
+  <xacro:macro name="wojtek_ros2_control" params="kp kd max_torque usb_port bus:=spi can_baud:=8 dry_run:=false tau_ff:=false link_timeout_cycles:=20">
     <ros2_control name="MD80HardwareInterface" type="system">
       <hardware>
@@ -60,4 +60,10 @@
              states still stream. Wired from the launches' dry_run arg. -->
         <param name="dry_run">${dry_run}</param>
+        <!-- Drive link watchdog: read() fails once any drive has delivered
+             no frame for more than this many controller cycles (20 = 100 ms
+             at the 200 Hz update_rate), and the controller manager drops
+             the component into on_error instead of streaming frozen states
+             as if the robot were alive. 0 = off. -->
+        <param name="link_timeout_cycles">${link_timeout_cycles}</param>
       </hardware>
       <xacro:wojtek_joint name="front_left_first_joint" can_id="10" kp="${kp}" kd="${kd}" max_torque="${max_torque}" tau_ff="${tau_ff}" />
